File: CC_dummy_load.sch (KiCad schematic (older format))
At the start: 54 parts, among them P1 CONN_01X02, P2 12vFAN, P3 CONN_01X09, P4 LOAD, Q1 Darl_NPN, Q2 IRF540N, U1 LM324N, U2 MCP4921-E/P, U3 LM35

Commit message: PCB first version
Parts:
- P1: footprint Pin_Headers:Pin_Header_Straight_1x02 -> Connect:bornier2
Changed lines of the file:
@@
 F 0 "P1" H 969 1168 50  0000 C CNN
 F 1 "CONN_01X02" H 969 1260 50  0000 C CNN
-F 2 "Pin_Headers:Pin_Header_Straight_1x02" H 1050 1450 50  0001 C CNN
+F 2 "Connect:bornier2" H 1050 1450 50  0001 C CNN
 F 3 "" H 1050 1450 50  0000 C CNN
 	1    1050 1450

Commit message: rev 2
Parts:
- removed P3: CONN_01X09, Pin_Headers:Pin_Header_Straight_1x09, symbol CONN_01X09
- removed RV1, RV3: POT, Potentiometers:Potentiometer_Trimmer-Suntan-TSR-3386P, symbol POT
- removed RV2: 10k, Potentiometers:Potentiometer_Trimmer-Suntan-TSR-3386P, symbol POT
- added C19: 150pF, Capacitors_ThroughHole:C_Disc_D3_P2.5, symbol C
- added P3: Arduino_Nano, arduino:Nano, symbol CONN_02X15
- added P5: KeyPad, Pin_Headers:Pin_Header_Straight_1x07, symbol CONN_01X07
- added P6: LCD_I2C, Pin_Headers:Pin_Header_Straight_1x04, symbol CONN_01X04
- added R21, R22: 9.09k, Resistors_ThroughHole:Resistor_Horizontal_RM10mm, symbol R
- added R23: 10k, Resistors_ThroughHole:Resistor_Horizontal_RM10mm, symbol R
- added R24, R26: 22k, Resistors_ThroughHole:Resistor_Horizontal_RM10mm, symbol R
- added R25: 3.3k, Resistors_ThroughHole:Resistor_Horizontal_RM10mm, symbol R
- added R27, R28: 6.8k, Resistors_ThroughHole:Resistor_Horizontal_RM10mm, symbol R
- added R29: 4.7k, Resistors_ThroughHole:Resistor_Horizontal_RM10mm, symbol R
- C16: value 100n -> 150pF; footprint Capacitors_ThroughHole:C_Disc_D6_P5 -> Capacitors_ThroughHole:C_Disc_D3_P2.5
- C17: value 22n -> 8.2nF
- C3, C4: value C -> 100n
- R12, R13, R14, R15, R17, R18, R19, R20, R7, R9: footprint Resistors_ThroughHole:Resistor_Horizontal_RM20mm -> Resistors_ThroughHole:Resistor_Horizontal_RM10mm
- R8: value 1k -> 2k
Connections:
- net ADC-VIN: now also R23.2
- net ARDU-A0: now also P3.19 (P19)
- net ARDU-P07: now also P3.6 (P6)
- net ARDU-P08: now also P3.5 (P5)
- net ARDU-P09: now also P3.4 (P4)
- net ARDU-P11: now also P3.2 (P2)
- net ARDU-P12: now also P3.1 (P1)
- net ARDU-P13: now also P3.16 (P16)
- net GND: now also C19.2, P3.12 (P12), P3.29 (P29), P5.4 (P4), P6.2 (P2), R29.2
- net at C16.1, R6.1, U1.12 (+): now also C19.1, R22.2
- net at U2.8 (VoutA): now also R22.1
- net at P4.1 (P1), Q2.2 (D), R16.1: now also R23.1
- net at R1.1, U1.6 (-): now also R21.2
- net at ADC1.3 (CH1), C10.1, C11.2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: now also R21.1
- net at D2.1 (K): now also P3.30 (P30)
- new net: P3.23 (P23), P6.3 (P3)
- new net: P3.24 (P24), P6.4 (P4)
- new net: P5.5 (P5), R24.1
- new net: P5.6 (P6), R24.2, R25.1
- new net: P5.1 (P1), R27.1
- new net: P5.2 (P2), R27.2, R28.1
- new net: P5.3 (P3), R28.2, R29.1
- new net ARDU-5v: P3.27 (P27), P6.1 (P1), R26.1
- new net ARDU-A1: P3.20 (P20), P5.7 (P7), R25.2, R26.2
- no-connect marks 4 -> 17
Other:
- note removed: "ARDU-GND"
- note removed: "ARDU-Vin"
- note removed: "Adjust the pot to create\na x10 amplification on Op-Amp\n(9k)"
- note removed: "Adjust the pot\nto divide VIN --> 4.096v\n(6.337k)"
- note removed: "Set the POT\nat 9.k\n(div /10)"
- moved on the sheet: C1, C16, C2, C5, C7, D2, P1, R1, U3, VR1
